Commit message: timely

File: urdf/fcs4hand2310.urdf (robot description, URDF)
Before this commit: robot fcs2310, 6 links, 5 joints
Links:
- removed link hub31x2
- added link hub71; visual box size=0.006 0.014 0.020; visual box size=0.020 0.062 0.014
Joints:
- joint hub: child hub31x2 -> hub71; origin xyz=0.013 0 0.040 rpy=0 1.57079632679489661923 0 -> xyz=0.013 0 0.041 rpy=0 1.57079632679489661923 0

File: urdf/fcs4hand2310ctrl.xacro (robot description, xacro)
@@ -1,6 +1,6 @@
 <?xml version="1.0"?>
-<robot name="fcs2310" xmlns:xacro="http://www.ros.org/wiki/xacro">
+<robot name="fcs4hand2310" xmlns:xacro="http://www.ros.org/wiki/xacro">
   <xacro:include filename="$(find fcs4hand2310)/urdf/fcs4hand2310.urdf"/>
-  <ros2_control name="fcs" type="system">
+  <ros2_control name="fcs0" type="system">
     <hardware>
       <plugin>hardware_fcs/HardwareFCS</plugin>
